File: pcb design/IGBT_board.sch (KiCad schematic (older format))
At the start: 51 parts, among them J1 4-794627-0, Q1 IGBT, Q10 IGBT, Q11 IGBT, Q12 IGBT, Q2 IGBT, Q3 IGBT, Q4 IGBT, Q5 IGBT, Q6 IGBT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

Commit message: Added NAND gates for shoot-through protection, and to configure the driver so when a fault is asserted the whole inverter will be shut down until a reset signal is issued
Signed-off-by: Marcos Chaparro <mchaparro@paltatech.com>
Parts:
- added C50: 100nF, IPC7351-Nominal:CAPC1608X55, symbol C-0603
- added U4: NAND, smd-semi:SOT-23-5, symbol 741G00-SOT23
Connections:
- net labels added: PWR_GOOD
- wire segments 167 -> 250
Other:
- note added: "HALF BRIDGE IGBT MODULE"
- note added: "Highest performance: IXXX200N65B4\nreasonable performance: IXXX110N65B4H1\ntesla used IKW75N60TFKSA1"
- note added: "If both PWM inputs are high,\nwe trigger the FAULT signal\nwhich turns off the whole\ninverter and will be latched\nuntil a reset is issued"
- note added: "The plan is to design it for 70kw continuous, 200kw peak\n\nSo, at 400v you need 175 Amp per phase (70kw x 2.5).\nThat is 30A per IGBT\n\nAt 30A, 0.9v Vce = 27W per transistor\n\nAt 45°C ambient temperature, if we want 75°C\nJunction temp, its a 30°C dT, and we need a\ntotal Rthja < 1.1°C/W\n\n0.15°C/W RthCS = thermal resistance,\ncase to heat sink (from the device data sheet). \n\n\n\n\n\n\n"
- note removed: "Highest performance: IXXX200N65B4\nFGY120T65S_F085 looks good but don't know about tab and heatsinking\ntesla used IKW75N60TFKSA1"
- note removed: "Specs are 200kw peak, 70kw continuous\n\nSo, at 400v you need 175 Amp per phase (70kw x 2.5). That is 30A per IGBT\n\nAt 30A, 0.9v Vce = 27W per transistor\n\nAt 45°C ambient temperature, if we want 75°C Junction temp, its a 30°C dT, and we need a total Rthja < 1.1°C/W\n\n0.15°C/W RthCS = thermal resistance, case to heat sink (from the device data sheet). \n\n\n\n\n\n\n"
- moved on the sheet: DS1, DS2, DS3, J1, MP1, Q1, Q10, Q11, Q12, Q2, Q3, Q4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

Commit message: Updated viable IGBT part#, selected infineon IGBT as project default
Signed-off-by: Marcos Chaparro <mchaparro@paltatech.com>
Parts:
- Q1: mfg# IXXX110N65B4H1 -> AUIRGPS4067D1
Other:
- note added: "Capacitors must be ably tu supply roughly 65% of battery\nsupplied current, so its important to have enough rms\ncurrent in the cap bank.\nIn this case, if we plan for 200kW at 500A, we should expect\na total RMS current of 325A in the capacitors.\nWe have 16uF*7*3 = 336uF\n14Arms per cap -> 98Arms per module, 296Arms per inverter"
- note added: "Highest performance: AUIRGPS4067D1\nreasonable performance: IXXX110N65B4H1\ntesla used IKW75N60TFKSA1"
- note removed: "Capacitors must be ably tu supply roughly 65% of battery\nsupplied current, so its important to have enough rms\ncurrent in the cap bank.\nIn this case, if we plan for 200kW at 500A, we should expect\na total RMS current of 325A in the capacitors.\nWe have 16uF*7*3 = 336uF"
- note removed: "Highest performance: IXXX200N65B4\nreasonable performance: IXXX110N65B4H1\ntesla used IKW75N60TFKSA1"
- note removed: "oxido y cobre"
Changed lines of the file:
@@
 Sheet 1 4
 Title "IGBT module"
-Date "2016-11-09"
+Date "2016-11-24"
 Rev "A"
 Comp "PALTA TECH S.A."
@@
 F 2 "pth-semi:TO-247" H 5627 3459 60  0001 L CNN
 F 3 "" H 5500 3600 60  0000 C CNN
-F 4 "IXXX110N65B4H1" H 5500 3550 60  0001 C CNN "mfg#"
+F 4 "AUIRGPS4067D1" H 5500 3550 60  0001 C CNN "mfg#"
 	1    5500 3550
 	1    0    0    -1
@@
 $EndComp
 Text Notes 600  6400 0    60   ~ 0
-Highest performance: IXXX200N65B4\nreasonable performance: IXXX110N65B4H1\ntesla used IKW75N60TFKSA1
+Highest performance: AUIRGPS4067D1\nreasonable performance: IXXX110N65B4H1\ntesla used IKW75N60TFKSA1
 $Comp
 L R-2512 R1
@@
 Text Notes 600  8300 0    60   ~ 0
 The plan is to design it for 70kw continuous, 200kw peak\n\nSo, at 400v you need 175 Amp per phase (70kw x 2.5).\nThat is 30A per IGBT\n\nAt 30A, 0.9v Vce = 27W per transistor\n\nAt 45°C ambient temperature, if we want 75°C\nJunction temp, its a 30°C dT, and we need a\ntotal Rthja < 1.1°C/W\n\n0.15°C/W RthCS = thermal resistance,\ncase to heat sink (from the device data sheet). \n\n\n\n\n\n\n
-Text Notes 5950 6350 0    60   ~ 0
+Text Notes 6950 6950 0    60   ~ 0
 Sil-pad thermal: SPK4-0.006-00-11.512
-Text Notes 9300 1650 0    40   ~ 0
-Capacitors must be ably tu supply roughly 65% of battery\nsupplied current, so its important to have enough rms\ncurrent in the cap bank.\nIn this case, if we plan for 200kW at 500A, we should expect\na total RMS current of 325A in the capacitors.\nWe have 16uF*7*3 = 336uF
-Text Notes 11350 3300 0    60   ~ 0
-oxido y cobre
+Text Notes 9250 1750 0    40   ~ 0
+Capacitors must be ably tu supply roughly 65% of battery\nsupplied current, so its important to have enough rms\ncurrent in the cap bank.\nIn this case, if we plan for 200kW at 500A, we should expect\na total RMS current of 325A in the capacitors.\nWe have 16uF*7*3 = 336uF\n14Arms per cap -> 98Arms per module, 296Arms per inverter
 $Sheet
 S 2950 2750 1350 950
