File: pcb design/IGBT_board.sch (KiCad schematic (older format))
At the start: 69 parts, among them J1 CONN-100MIL-M-2x8, J5 PHASE CURRENT CONN, Q1 IGBT, Q10 IGBT, Q11 IGBT, Q12 IGBT, Q2 IGBT, Q3 IGBT, Q4 IGBT, Q5 IGBT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

Commit message: Add gate driver load to enable 2 step turnoff in buffered configuration. Updated layout.
Signed-off-by: Marcos Chaparro <mchaparro@paltatech.com>
Parts:
- removed DS4: CAPS_CHARGED, smd-semi:LED-0603, symbol LED-0603
- removed R62, R63, R66: 50k 1W, IPC7351-Nominal:RESC6432X70, symbol R-2512
- C1, C2, C3, C4, C5, C6, C7: symbol C-FILM-6mm -> pasv-cap:C-FILM-6mm; MPN (none) -> B32796G3166K
- C51, C52: symbol C-0805 -> pasv-cap:C-0805
- C77, C82, C85: symbol C-0603 -> pasv-cap:C-0603
- D19: symbol TVS_BI -> _semi:TVS_BI; MPN (none) -> SMBJ24A
- DS1, DS2, DS3: symbol LED-0603 -> semi-opto-generic:LED-0603
- F1: symbol FUSE -> _passive:FUSE; MPN (none) -> 0ZCJ0050AF2E
- J1: symbol CONN-100MIL-M-2x8 -> conn-100mil:CONN-100MIL-M-2x8
- J5: symbol CONN-100MIL-M-1x4 -> conn-100mil:CONN-100MIL-M-1x4
- MP1: symbol HEATSINK-NO-CONN -> mechanical1:HEATSINK-NO-CONN
- Q1: symbol IGBT -> _semi:IGBT; MPN (none) -> IXXX110N65B4H1; mfg# AUIRGPS4067D1 -> IXXX110N65B4H1
- Q10, Q11, Q12, Q2, Q3, Q4, Q5, Q6, Q7, Q8, Q9: symbol IGBT -> _semi:IGBT; MPN (none) -> IXXX110N65B4H1
- R1, R2: value 20R -> 1R; symbol R-2512 -> pasv-res:R-2512; Exclude from BOM (none) -> 0; mfg# CRCW251220R0FKEG -> (none)
- R10, R11, R12, R13, R14, R15, R16, R17, R18, R19, R20, R21, R22, R23, R24, R3, R4, R5, R6, R7, R8, R9: symbol R-2512 -> pasv-res:R-2512; MPN (none) -> CRCW251220R0FKEG
- R51, R52, R53, R54, R56, R59, R61: symbol R-0603 -> pasv-res:R-0603
- SYM1: symbol OSHW-SCHEM-PCB10mm -> symbol:OSHW-SCHEM-PCB10mm; version (none) -> none
- U5: symbol LM1117IMP-v.v -> TexasInstruments:LM1117IMP-v.v
Other:
- note added: "Rg < Rgdriver / N / 10\nfor lower Rg mismatch"
- note added: "Use common\nmode chokes?"
- note removed: "Bleeding R's"
