File: pcb design/IGBT_driver.sch (KiCad schematic (older format))
At the start: 38 parts, among them J2 DESAT, Q13 NPN, Q14 PNP, U1 ISO5852S

Commit message: Added NAND gates for shoot-through protection, and to configure the driver so when a fault is asserted the whole inverter will be shut down until a reset signal is issued
Signed-off-by: Marcos Chaparro <mchaparro@paltatech.com>
Parts:
- removed U?: SN74AUC1G14, smd-semi:SOT-23-5, symbol 741G04-SOT23
- added C?: 100nF, IPC7351-Nominal:CAPC1608X55, symbol C-0603
- added U? (x2): NAND, smd-semi:SOT-23-5, symbol 741G00-SOT23
- gave numbers to parts that had none: 1
Connections:
- wire segments 84 -> 90
Other:
- moved on the sheet: TP3
Changed lines of the file:
@@
 -8V
 $Comp
-L GND #PWR03
+L GND #PWR04
 U 1 1 58241AEC
 P 3150 4050
-AR Path="/5822D62D/58241AEC" Ref="#PWR03"  Part="1"
-AR Path="/5824556D/58241AEC" Ref="#PWR019"  Part="1"
-F 0 "#PWR03" H 3150 4050 30  0001 C CNN
+AR Path="/5822D62D/58241AEC" Ref="#PWR04"  Part="1"
+AR Path="/5824556D/58241AEC" Ref="#PWR021"  Part="1"
+F 0 "#PWR04" H 3150 4050 30  0001 C CNN
 F 1 "GND" H 3150 3980 30  0001 C CNN
 F 2 "" H 3150 4050 60  0000 C CNN
@@
 $EndComp
 $Comp
-L GND #PWR04
+L GND #PWR05
 U 1 1 5830FC3F
 P 1950 4000
-AR Path="/5822D62D/5830FC3F" Ref="#PWR04"  Part="1"
-AR Path="/5824556D/5830FC3F" Ref="#PWR020"  Part="1"
-F 0 "#PWR04" H 1950 4000 30  0001 C CNN
+AR Path="/5822D62D/5830FC3F" Ref="#PWR05"  Part="1"
+AR Path="/5824556D/5830FC3F" Ref="#PWR022"  Part="1"
+F 0 "#PWR05" H 1950 4000 30  0001 C CNN
 F 1 "GND" H 1950 3930 30  0001 C CNN
 F 2 "" H 1950 4000 60  0000 C CNN
@@
 	0    -1   -1   0
 $EndComp
-Text GLabel 2300 4050 2    50   Input ~ 0
-3.3v
-Text HLabel 800  4300 0    60   Input ~ 0
+Text HLabel 750  4300 0    60   Input ~ 0
 IN+
 Text Notes 900  4400 2    30   ~ 0
@@
 L TESTPOINT TP?
 U 1 1 58364308
-P 1950 4300
+P 850 4200
 AR Path="/58232371/58364308" Ref="TP?"  Part="1"
 AR Path="/5822D62D/58364308" Ref="TP3"  Part="1"
 AR Path="/5824556D/58364308" Ref="TP13"  Part="1"
-F 0 "TP3" H 2010 4421 50  0000 L CNN
-F 1 "IN" H 2010 4330 50  0000 L CNN
-F 2 "conn-test:TEST-SMD-SMALL" H 1950 4300 50  0001 C CNN
-F 3 "" H 1950 4300 50  0000 C CNN
-	1    1950 4300
-	1    0    0    1
+F 0 "TP3" H 910 4321 50  0000 L CNN
+F 1 "IN" H 910 4230 50  0000 L CNN
+F 2 "conn-test:TEST-SMD-SMALL" H 850 4200 50  0001 C CNN
+F 3 "" H 850 4200 50  0000 C CNN
+	1    850  4200
+	-1   0    0    -1
 $EndComp
 $Comp
@@
 P 3450 5250
 AR Path="/5822D62D/58363068" Ref="#PWR06"  Part="1"
-AR Path="/5824556D/58363068" Ref="#PWR022"  Part="1"
+AR Path="/5824556D/58363068" Ref="#PWR023"  Part="1"
 F 0 "#PWR06" H 3450 5250 30  0001 C CNN
 F 1 "GND" H 3450 5180 30  0001 C CNN
@@
 TH to connect to\ncopper collector layer
 Connection ~ 3000 4700
-$Comp
-L 741G04-SOT23 U?
-U 1 1 58362FBD
-P 2300 4300
-F 0 "U?" H 2350 4400 50  0000 L CNN
-F 1 "SN74AUC1G14" H 2400 4200 50  0000 L CNN
-F 2 "smd-semi:SOT-23-5" H 2300 4300 50  0001 C CNN
-F 3 "" H 2150 4550 60  0000 C CNN
-F 4 "SN74AUC1G14DBVR" H 2300 4300 60  0001 C CNN "mfg#"
-	1    2300 4300
-	1    0    0    -1
-$EndComp
-Wire Wire Line
-	2300 4050 2250 4050
-Wire Wire Line
-	2250 4050 2250 4150
-$Comp
-L GND #PWR?
-U 1 1 58363902
-P 2250 4450
-AR Path="/5822D62D/58363902" Ref="#PWR?"  Part="1"
-AR Path="/5824556D/58363902" Ref="#PWR?"  Part="1"
-F 0 "#PWR?" H 2250 4450 30  0001 C CNN
-F 1 "GND" H 2250 4380 30  0001 C CNN
-F 2 "" H 2250 4450 60  0000 C CNN
-F 3 "" H 2250 4450 60  0000 C CNN
-	1    2250 4450
-	1    0    0    -1
-$EndComp
 Wire Wire Line
-	800  4300 2050 4300
-Connection ~ 1950 4300
+	750  4300 1950 4300
 Connection ~ 900  4300
 $Comp
-L GND #PWR?
+L GND #PWR08
 U 1 1 583666D4
 P 1000 4550
-AR Path="/5822D62D/583666D4" Ref="#PWR?"  Part="1"
-AR Path="/5824556D/583666D4" Ref="#PWR?"  Part="1"
-F 0 "#PWR?" H 1000 4550 30  0001 C CNN
+AR Path="/5822D62D/583666D4" Ref="#PWR08"  Part="1"
+AR Path="/5824556D/583666D4" Ref="#PWR025"  Part="1"
+F 0 "#PWR08" H 1000 4550 30  0001 C CNN
 F 1 "GND" H 1000 4480 30  0001 C CNN
 F 2 "" H 1000 4550 60  0000 C CNN
@@
 	1    0    0    -1
 $EndComp
-Text GLabel 950  4000 0    50   Input ~ 0
+Text GLabel 950  3850 0    50   Input ~ 0
 3.3v
 Wire Wire Line
-	950  4000 1000 4000
+	950  3850 1000 3850
 Wire Wire Line
-	1000 4000 1000 4050
+	1000 3850 1000 4050
 $Comp
-L R-0603 R?
+L R-0603 R28
 U 1 1 5836826A
 P 1900 5100
-AR Path="/5822D62D/5836826A" Ref="R?"  Part="1"
-AR Path="/5824556D/5836826A" Ref="R?"  Part="1"
-F 0 "R?" V 1700 5100 50  0000 C CNN
+AR Path="/5822D62D/5836826A" Ref="R28"  Part="1"
+AR Path="/5824556D/5836826A" Ref="R45"  Part="1"
+F 0 "R28" V 1700 5100 50  0000 C CNN
 F 1 "10k" V 1800 5100 50  0000 C CNN
 F 2 "IPC7351-Nominal:RESC1608X50" H 1900 5100 50  0001 C CNN
@@
 $EndComp
 $Comp
-L GND #PWR?
+L GND #PWR09
 U 1 1 58368450
 P 1900 5250
-AR Path="/5822D62D/58368450" Ref="#PWR?"  Part="1"
-AR Path="/5824556D/58368450" Ref="#PWR?"  Part="1"
-F 0 "#PWR?" H 1900 5250 30  0001 C CNN
+AR Path="/5822D62D/58368450" Ref="#PWR09"  Part="1"
+AR Path="/5824556D/58368450" Ref="#PWR026"  Part="1"
+F 0 "#PWR09" H 1900 5250 30  0001 C CNN
 F 1 "GND" H 1900 5180 30  0001 C CNN
 F 2 "" H 1900 5250 60  0000 C CNN
@@
 	1900 4300 1900 5000
 Connection ~ 1900 4300
+Wire Wire Line
+	1950 4350 2000 4350
+Wire Wire Line
+	1950 4250 1950 4350
+Wire Wire Line
+	2000 4250 1950 4250
+Connection ~ 1950 4300
+Wire Wire Line
+	850  4200 850  4300
+Connection ~ 850  4300
+$Comp
+L 741G00-SOT23 U?
+U 2 1 58394A62
+P 2650 5450
+F 0 "U?" H 2730 5196 50  0000 L CNN
+F 1 "NAND" H 2730 5105 50  0000 L CNN
+F 2 "smd-semi:SOT-23-5" H 2650 5300 50  0001 C CNN
+F 3 "" H 2450 5450 60  0000 C CNN
+F 4 "SN74LVC1G38DBVR" H 2650 5450 60  0001 C CNN "mfg#"
+	2    2650 5450
+	1    0    0    -1
+$EndComp
+$Comp
+L 741G00-SOT23 U?
+U 1 1 58394A6A
+P 2350 4300
+AR Path="/58394A6A" Ref="U?"  Part="1"
+AR Path="/5822D62D/58394A6A" Ref="U?"  Part="1"
+F 0 "U?" H 2300 4575 50  0000 C CNN
+F 1 "NAND" H 2300 4484 50  0000 C CNN
+F 2 "smd-semi:SOT-23-5" H 2350 4150 50  0001 C CNN
+F 3 "" H 2150 4300 60  0000 C CNN
+F 4 "SN74LVC1G38DBVR" H 2350 4300 60  0001 C CNN "mfg#"
+	1    2350 4300
+	1    0    0    -1
+$EndComp
+$Comp
+L C-0603 C?
+U 1 1 58394A72
+P 2450 5750
+F 0 "C?" H 2562 5796 50  0000 L CNN
+F 1 "100nF" H 2562 5705 50  0000 L CNN
+F 2 "IPC7351-Nominal:CAPC1608X55" H 2450 5750 50  0001 C CNN
+F 3 "" H 2440 5725 60  0000 C CNN
+F 4 "CAP MLCC 100pF C0G 50V 5% [0603]" H 3250 6300 60  0001 C CNN "BOM"
+	1    2450 5750
+	-1   0    0    -1
+$EndComp
+Wire Wire Line
+	2400 5500 2650 5500
+Wire Wire Line
+	2450 5500 2450 5650
+Wire Wire Line
+	2650 6000 2450 6000
+Wire Wire Line
+	2450 5850 2450 6050
+$Comp
+L GND #PWR?
+U 1 1 58394A7D
+P 2450 6050
+F 0 "#PWR?" H 2450 6050 30  0001 C CNN
+F 1 "GND" H 2450 5980 30  0001 C CNN
+F 2 "" H 2450 6050 60  0000 C CNN
+F 3 "" H 2450 6050 60  0000 C CNN
+	1    2450 6050
+	1    0    0    -1
+$EndComp
+Connection ~ 2450 6000
+Text GLabel 2400 5500 0    50   Input ~ 0
+3.3v
+Connection ~ 2450 5500
 $EndSCHEMATC

Commit message: Updated viable IGBT part#, selected infineon IGBT as project default
Signed-off-by: Marcos Chaparro <mchaparro@paltatech.com>
Changed lines of the file:
@@
 Wire Notes Line
 	4350 5900 4350 2750
-Wire Notes Line
-	4350 5900 11700 5900
-Wire Notes Line
-	3850 2750 11200 2750
 Wire Wire Line
 	1950 3750 1950 3700
@@
 U 2 1 58394A62
 P 2650 5450
+AR Path="/5822D62D/58394A62" Ref="U?"  Part="2"
+AR Path="/5824556D/58394A62" Ref="U?"  Part="2"
 F 0 "U?" H 2730 5196 50  0000 L CNN
 F 1 "NAND" H 2730 5105 50  0000 L CNN
@@
 AR Path="/58394A6A" Ref="U?"  Part="1"
 AR Path="/5822D62D/58394A6A" Ref="U?"  Part="1"
+AR Path="/5824556D/58394A6A" Ref="U?"  Part="1"
 F 0 "U?" H 2300 4575 50  0000 C CNN
 F 1 "NAND" H 2300 4484 50  0000 C CNN
@@
 U 1 1 58394A72
 P 2450 5750
+AR Path="/5822D62D/58394A72" Ref="C?"  Part="1"
+AR Path="/5824556D/58394A72" Ref="C?"  Part="1"
 F 0 "C?" H 2562 5796 50  0000 L CNN
 F 1 "100nF" H 2562 5705 50  0000 L CNN
@@
 U 1 1 58394A7D
 P 2450 6050
+AR Path="/5822D62D/58394A7D" Ref="#PWR?"  Part="1"
+AR Path="/5824556D/58394A7D" Ref="#PWR?"  Part="1"
 F 0 "#PWR?" H 2450 6050 30  0001 C CNN
 F 1 "GND" H 2450 5980 30  0001 C CNN
@@
 3.3v
 Connection ~ 2450 5500
+Wire Notes Line
+	4350 2750 11200 2750
+Wire Notes Line
+	11200 5900 4350 5900
 $EndSCHEMATC
