File: pcb design/IGBT_driver_power_suply.sch (KiCad schematic (older format))
At the start: 53 parts, among them Q15 CSD19533Q5A, Q16 CSD19533Q5A, T1 TRANS-3-1CT, U2 LM5030

Commit message: Changed isolated amplifier from AMC1200 to AMC1301 because it has reinforced isolation. This required a different layout
Signed-off-by: Marcos Chaparro <mchaparro@paltatech.com>
Changed lines of the file:
@@
 $EndComp
 Wire Wire Line
-	2950 3150 2950 3250
-Wire Wire Line
-	2950 3250 2950 3300
+	2950 3150 2950 3300
 Wire Wire Line
 	3200 3300 3200 3250
 Wire Wire Line
-	2950 3250 3200 3250
-Wire Wire Line
-	3200 3250 3400 3250
+	2950 3250 3400 3250
 Connection ~ 2950 3250
 Wire Wire Line
@@
 	2250 4450 2250 4350
 Wire Wire Line
-	1600 3550 1600 4150
-Wire Wire Line
-	1600 4150 1600 4350
+	1600 3550 1600 4350
 Wire Wire Line
 	1600 4150 2250 4150
@@
 	4100 4300 4850 4300
 Wire Wire Line
-	4450 4000 4450 4100
-Wire Wire Line
-	4450 4100 4450 4500
-Wire Wire Line
-	4450 4500 4450 4750
-Wire Wire Line
-	4450 4750 4450 4850
-Wire Wire Line
-	4450 4500 4950 4500
-Wire Wire Line
-	4950 4500 5000 4500
-Wire Wire Line
-	5000 4500 5050 4500
+	4450 4000 4450 4850
+Wire Wire Line
+	4450 4500 5050 4500
 Wire Wire Line
 	4950 4500 4950 4350
@@
 	4500 4000 4500 4100
 Wire Wire Line
-	4450 4100 4500 4100
-Wire Wire Line
-	4500 4100 4550 4100
+	4450 4100 4550 4100
 Connection ~ 4450 4100
 Wire Wire Line
@@
 	2950 2750 2700 2750
 Wire Wire Line
-	4600 3550 5350 3550
-Wire Wire Line
-	5350 3550 6000 3550
-Wire Wire Line
-	4600 3550 4600 3700
-Wire Wire Line
-	4600 3700 4600 3800
+	4600 3550 6000 3550
+Wire Wire Line
+	4600 3550 4600 3800
 Wire Wire Line
 	4550 3700 4550 3800
 Wire Wire Line
-	4450 3700 4500 3700
-Wire Wire Line
-	4500 3700 4550 3700
-Wire Wire Line
-	4550 3700 4600 3700
+	4450 3700 4600 3700
 Connection ~ 4600 3700
 Wire Wire Line
@@
 Connection ~ 4500 3700
 Wire Wire Line
-	5100 3750 5450 3750
-Wire Wire Line
-	5450 3750 6000 3750
-Wire Wire Line
-	5100 3750 5100 4050
-Wire Wire Line
-	5100 4050 5100 4150
+	5100 3750 6000 3750
+Wire Wire Line
+	5100 3750 5100 4150
 Wire Wire Line
 	5050 4050 5050 4150
 Wire Wire Line
-	4950 4050 5000 4050
-Wire Wire Line
-	5000 4050 5050 4050
-Wire Wire Line
-	5050 4050 5100 4050
+	4950 4050 5100 4050
 Connection ~ 5100 4050
 Wire Wire Line
@@
 	1200 4350 1200 4050
 Wire Wire Line
-	1150 4050 1200 4050
-Wire Wire Line
-	1200 4050 2250 4050
+	1150 4050 2250 4050
 Connection ~ 1200 4050
 Wire Wire Line
 	850  4050 950  4050
 Wire Wire Line
-	1200 4550 1200 4600
-Wire Wire Line
-	1200 4600 1200 4650
+	1200 4550 1200 4650
 Wire Wire Line
 	1600 4650 1600 4550
@@
 	6300 3200 6300 3050
 Wire Wire Line
-	6300 3050 7300 3050
-Wire Wire Line
-	7300 3050 8250 3050
-Wire Wire Line
-	8250 3050 8850 3050
-Wire Wire Line
-	8850 3050 9500 3050
-Wire Wire Line
-	9500 3050 10100 3050
-Wire Wire Line
-	10100 3050 10400 3050
+	6300 3050 10400 3050
 $Comp
 L C-1206 C25
@@
 	8250 3550 8250 3800
 Wire Wire Line
-	7300 3800 8250 3800
-Wire Wire Line
-	8250 3800 8850 3800
-Wire Wire Line
-	8850 3800 9500 3800
-Wire Wire Line
-	9500 3800 10100 3800
-Wire Wire Line
-	10100 3800 10400 3800
-Wire Wire Line
-	8250 2750 8250 3050
-Wire Wire Line
-	8250 3050 8250 3350
+	7300 3800 10400 3800
+Wire Wire Line
+	8250 2750 8250 3350
 Connection ~ 8250 3050
 $Comp
@@
 Connection ~ 8250 3800
 Wire Wire Line
-	8850 2750 8850 3050
-Wire Wire Line
-	8850 3050 8850 3350
+	8850 2750 8850 3350
 Connection ~ 8850 3050
 $Comp
@@
 Connection ~ 8850 3800
 Wire Wire Line
-	9500 2750 9500 3050
-Wire Wire Line
-	9500 3050 9500 3350
+	9500 2750 9500 3350
 Connection ~ 9500 3050
 $Comp
@@
 $EndComp
 Wire Wire Line
-	7300 2900 7300 3050
-Wire Wire Line
-	7300 3050 7300 3200
+	7300 2900 7300 3200
 Connection ~ 7300 3050
 $Comp
@@
 $EndComp
 Wire Wire Line
-	7300 2600 7300 2650
-Wire Wire Line
-	7300 2650 7300 2700
+	7300 2600 7300 2700
 Wire Wire Line
 	7300 2650 7100 2650
@@
 	7300 2400 7300 2300
 Wire Wire Line
-	7300 2300 8250 2300
-Wire Wire Line
-	8250 2300 8850 2300
-Wire Wire Line
-	8850 2300 9500 2300
-Wire Wire Line
-	9500 2300 10100 2300
-Wire Wire Line
-	10100 2300 10400 2300
+	7300 2300 10400 2300
 Wire Wire Line
 	8250 2300 8250 2550
@@
 $EndComp
 Wire Wire Line
-	6300 5150 7300 5150
-Wire Wire Line
-	7300 5150 8250 5150
-Wire Wire Line
-	8250 5150 8850 5150
-Wire Wire Line
-	8850 5150 9500 5150
-Wire Wire Line
-	9500 5150 10100 5150
-Wire Wire Line
-	10100 5150 10400 5150
-Wire Wire Line
-	6300 5550 6800 5550
-Wire Wire Line
-	6800 5550 6900 5550
+	6300 5150 10400 5150
+Wire Wire Line
+	6300 5550 6900 5550
 $Comp
 L C-1206 C27
@@
 	8250 5650 8250 5900
 Wire Wire Line
-	7300 5900 8250 5900
-Wire Wire Line
-	8250 5900 8850 5900
-Wire Wire Line
-	8850 5900 9500 5900
-Wire Wire Line
-	9500 5900 10100 5900
-Wire Wire Line
-	10100 5900 10400 5900
-Wire Wire Line
-	8250 4850 8250 5150
-Wire Wire Line
-	8250 5150 8250 5450
+	7300 5900 10400 5900
+Wire Wire Line
+	8250 4850 8250 5450
 Connection ~ 8250 5150
 $Comp
@@
 Connection ~ 8250 5900
 Wire Wire Line
-	8850 4850 8850 5150
-Wire Wire Line
-	8850 5150 8850 5450
+	8850 4850 8850 5450
 Connection ~ 8850 5150
 $Comp
@@
 Connection ~ 8850 5900
 Wire Wire Line
-	9500 4850 9500 5150
-Wire Wire Line
-	9500 5150 9500 5450
+	9500 4850 9500 5450
 Connection ~ 9500 5150
 $Comp
@@
 $EndComp
 Wire Wire Line
-	7300 5000 7300 5150
-Wire Wire Line
-	7300 5150 7300 5300
+	7300 5000 7300 5300
 Connection ~ 7300 5150
 $Comp
@@
 $EndComp
 Wire Wire Line
-	7300 4700 7300 4750
-Wire Wire Line
-	7300 4750 7300 4800
+	7300 4700 7300 4800
 Wire Wire Line
 	7300 4750 7100 4750
@@
 	7300 4500 7300 4400
 Wire Wire Line
-	7300 4400 8250 4400
-Wire Wire Line
-	8250 4400 8850 4400
-Wire Wire Line
-	8850 4400 9500 4400
-Wire Wire Line
-	9500 4400 10100 4400
-Wire Wire Line
-	10100 4400 10400 4400
+	7300 4400 10400 4400
 Wire Wire Line
 	8250 4400 8250 4650
@@
 	5900 3650 5950 3650
 Wire Wire Line
-	5900 2750 5900 2800
-Wire Wire Line
-	5900 2800 5900 3650
+	5900 2750 5900 3650
 $Comp
 L C-ALUM-6.3mm C45
@@
 $EndComp
 Wire Wire Line
-	5550 2800 5650 2800
-Wire Wire Line
-	5650 2800 5900 2800
+	5550 2800 5900 2800
 Wire Wire Line
 	5650 2800 5650 2900
@@
 	7300 3800 7300 3700
 Wire Wire Line
-	7300 3400 7300 3450
-Wire Wire Line
-	7300 3450 7300 3500
+	7300 3400 7300 3500
 $Comp
 L C-1206 C53
@@
 $EndComp
 Wire Wire Line
-	6300 3450 6800 3450
-Wire Wire Line
-	6800 3450 6900 3450
+	6300 3450 6900 3450
 Connection ~ 6800 3450
 Wire Wire Line
@@
 	7100 5550 7300 5550
 Wire Wire Line
-	7300 5500 7300 5550
-Wire Wire Line
-	7300 5550 7300 5600
+	7300 5500 7300 5600
 Connection ~ 7300 5550
 Wire Wire Line
