File: pcb design/phase_voltage_sensor.sch (KiCad schematic (older format))
At the start: 16 parts

Commit message: Connected phase sensing, added images
Signed-off-by: Marcos Chaparro <mchaparro@paltatech.com>
Other:
- note added: "0-800V phase voltage measurement\nwith isolation amplifier"
- note removed: "0-800V isolated phase voltage measurement"

Commit message: Phase voltage sensing laid out
Signed-off-by: Marcos Chaparro <mchaparro@paltatech.com>
Parts:
- removed C?: 1uF, IPC7351-Nominal:CAPC3216X70, symbol C-1206
- removed R? (x2): 500k, IPC7351-Nominal:RESC3216X60, symbol R-1206
- added J4: PHASE, conn-100mil:CONN-100MIL-F-1x1, symbol CONN-100MIL-F-1x1
- R82, R84: renamed from R?; value 500k -> 1M; #mfg (none) -> CHV1206-FX-1004ELF
- U10: renamed from U?; footprint IPC7351-Most:SOIC127P1032X265-8 -> IPC7351-Nominal:SOIC127P1032X265-8
- gave numbers to parts that had none: 10
Connections:
- net Vin+: now also R82.2, J4.1
- net VIN+: now reaches C79.1, R87.1, U10.2 (VINP)
- net VIN-: now reaches C79.2, R88.2, U10.3 (VINN)
Other:
- note added: "0-650V phase voltage measurement\nwith isolation amplifier"
- note added: "=1000/(2000000+11000)*650*8 = 2.58V differential output at 650V"
- note added: "These particular 1206\nresistors are rated at 800V each.\nPut slots though"
- note removed: "0-800V phase voltage measurement\nwith isolation amplifier"
- note removed: "1206 resistors are\nrated at 200V each"
- note removed: "=1000/(2000000+11000)*800*8 = 3.18V differential output"

Commit message: Updated gate resistor rating, qty and part#, updated desat blocking diode with much beetter recovery time
Signed-off-by: Marcos Chaparro <mchaparro@paltatech.com>
Other:
- note added: "0-650V phase voltage measurement\nusing isolation amplifier"
- note removed: "0-650V phase voltage measurement\nwith isolation amplifier"
Changed lines of the file:
@@
 These particular 1206\nresistors are rated at 800V each.\nPut slots though
 Text Notes 900  1550 0    260  ~ 52
-0-650V phase voltage measurement\nwith isolation amplifier
+0-650V phase voltage measurement\nusing isolation amplifier
 $Comp
 L BZX84 DZ6

Commit message: Changed isolated amplifier from AMC1200 to AMC1301 because it has reinforced isolation. This required a different layout
Signed-off-by: Marcos Chaparro <mchaparro@paltatech.com>
Parts:
- removed R86: 10k, IPC7351-Nominal:RESC1608X50, symbol R-0603
- removed R87: 12R, IPC7351-Nominal:RESC1608X50, symbol R-0603
- C78: footprint IPC7351-Nominal:CAPC3216X70 -> IPC7351-Nominal:CAPC1608X55
- C80: footprint IPC7351-Nominal:CAPC3216X70 -> IPC7351-Nominal:CAPC1608X55; BOM CAP MLCC 100pF C0G 50V 5% [1206] -> CAP MLCC 100pF C0G 50V 5% [0603]
- C81: value 1uF -> 2.2uF; footprint IPC7351-Nominal:CAPC3216X70 -> IPC7351-Nominal:CAPC1608X55; BOM CAP MLCC 100pF C0G 50V 5% [1206] -> CAP MLCC 100pF C0G 50V 5% [0603]
- R88: value 12R -> 1k
- U10: value AMC1200 -> AMC1301; #mfg AMC1200TDWVRQ1 -> AMC1301DWVR
Connections:
- net VIN+: now also R84.1, R85.1
- net Vin-: now also R85.2, R88.1
Other:
- note added: "=1000/(2000000+2000)*650*8.2 = 2.66V differential output at 650V"
- note removed: "=1000/(2000000+11000)*650*8 = 2.58V differential output at 650V"

Commit message: Add gate driver load to enable 2 step turnoff in buffered configuration. Updated layout.
Signed-off-by: Marcos Chaparro <mchaparro@paltatech.com>
Parts:
- C78: symbol C-1206 -> pasv-cap:C-1206; BOM CAP MLCC 100pF C0G 50V 5% [1206] -> CAP MLCC 100pF C0G 50V 5% [0603]
- C79: symbol C-0603 -> pasv-cap:C-0603
- C80, C81: symbol C-1206 -> pasv-cap:C-1206
- DZ6: symbol BZX84 -> semi-diode-generic:BZX84; MPN (none) -> BZX84-A5V1,215
- J4: symbol CONN-100MIL-F-1x1 -> conn-100mil:CONN-100MIL-F-1x1
- R82, R84: symbol R-1206 -> pasv-res:R-1206; MPN (none) -> CHV1206-FX-1004ELF
- R83, R85, R88: symbol R-0603 -> pasv-res:R-0603
- U10: symbol AMC1200 -> IGBT_board-rescue:AMC1200-RESCUE-IGBT_board; MPN (none) -> AMC1301DWVR
Other:
- note added: "Route very\nclose together"
Changed lines of the file:
@@
-EESchema Schematic File Version 2
-LIBS:Abracon
-LIBS:ActiveSemi
-LIBS:Altera
-LIBS:AMS
-LIBS:AnalogDevices
-LIBS:AOS
-LIBS:Atmel
-LIBS:Bosch
-LIBS:conn-100mil
-LIBS:conn-2mm
-LIBS:conn-amphenol
-LIBS:conn-assmann
-LIBS:conn-cui
-LIBS:conn-fci
-LIBS:conn-jae
-LIBS:conn-linx
-LIBS:conn-molex
-LIBS:conn-tagconnect
-LIBS:conn-te
-LIBS:conn-test
-LIBS:DiodesInc
-LIBS:display
-LIBS:electomech-misc
-LIBS:_electromech
-LIBS:Fairchild
-LIBS:FTDI
-LIBS:Infineon
-LIBS:Intersil
-LIBS:Lattice
-LIBS:_linear
-LIBS:LinearTech
-LIBS:Littelfuse
-LIBS:logic-4000
-LIBS:logic-7400
-LIBS:logic-7400-new
-LIBS:_logic
-LIBS:MACOM
-LIBS:Macrofab
-LIBS:maxim
-LIBS:mechanical
-LIBS:Microchip
-LIBS:Micron
-LIBS:Murata
-LIBS:NXP
-LIBS:OceanOptics
-LIBS:onsemi
-LIBS:_passive
-LIBS:pasv-BelFuse
-LIBS:pasv-BiTech
-LIBS:pasv-Bourns
-LIBS:pasv-cap
-LIBS:pasv-ind
-LIBS:pasv-Murata
-LIBS:pasv-res
-LIBS:pasv-TDK
-LIBS:pasv-xtal
-LIBS:pcb
-LIBS:power
-LIBS:Recom
-LIBS:Richtek
-LIBS:semi-diode-DiodesInc
-LIBS:semi-diode-generic
-LIBS:semi-diode-MCC
-LIBS:semi-diode-NXP
-LIBS:semi-diode-OnSemi
-LIBS:semi-diode-Semtech
-LIBS:semi-diode-ST
-LIBS:semi-diode-Toshiba
-LIBS:_semi
-LIBS:semi-opto-generic
-LIBS:semi-opto-liteon
-LIBS:semi-thyristor-generic
-LIBS:semi-trans-AOS
-LIBS:semi-trans-DiodesInc
-LIBS:semi-trans-EPC
-LIBS:semi-trans-Fairchild
-LIBS:semi-trans-generic
-LIBS:semi-trans-Infineon
-LIBS:semi-trans-IRF
-LIBS:semi-trans-IXYS
-LIBS:semi-trans-NXP
-LIBS:semi-trans-OnSemi
-LIBS:semi-trans-Panasonic
-LIBS:semi-trans-ST
-LIBS:semi-trans-TI
-LIBS:semi-trans-Toshiba
-LIBS:semi-trans-Vishay
-LIBS:silabs
-LIBS:skyworks
-LIBS:st_ic
-LIBS:ST
-LIBS:supertex
-LIBS:symbol
-LIBS:TexasInstruments
-LIBS:u-blox
-LIBS:Vishay
-LIBS:Winbond
-LIBS:Xilinx
-LIBS:paltatech
+EESchema Schematic File Version 4
 LIBS:IGBT_board-cache
 EELAYER 26 0
@@
 VDD2
 $Comp
-L C-1206 C78
+L pasv-cap:C-1206 C78
 U 1 1 585AE04F
 P 5100 3600
@@
 F 2 "IPC7351-Nominal:CAPC1608X55" H 5100 3600 50  0001 C CNN
 F 3 "" H 5090 3575 60  0000 C CNN
-F 4 "CAP MLCC 100pF C0G 50V 5% [1206]" H 5900 4150 60  0001 C CNN "BOM"
+F 4 "CAP MLCC 100pF C0G 50V 5% [0603]" H 5900 4150 60  0001 C CNN "BOM"
 	1    5100 3600
 	1    0    0    1
 $EndComp
 $Comp
-L AMC1200 U10
+L IGBT_board-rescue:AMC1200-RESCUE-IGBT_board U10
 U 1 1 585AEFF8
 P 5900 3850
+AR Path="/585AEFF8" Ref="U10"  Part="1"
+AR Path="/585ACB8D/585AEFF8" Ref="U10"  Part="1"
 F 0 "U10" H 5900 4537 60  0000 C CNN
 F 1 "AMC1301" H 5900 4431 60  0000 C CNN
@@
 F 3 "" H 5900 3850 60  0001 C CNN
 F 4 "AMC1301DWVR" H 6000 3400 60  0001 C CNN "#mfg"
+F 5 "AMC1301DWVR" H 0   0   60  0001 C CNN "MPN"
 	1    5900 3850
 	1    0    0    -1
@@
 Connection ~ 5100 3450
 $Comp
-L C-0603 C79
+L pasv-cap:C-0603 C79
 U 1 1 585AF5E7
 P 5100 4100
@@
 Connection ~ 5100 4250
 $Comp
-L R-0603 R88
+L pasv-res:R-0603 R88
 U 1 1 585AF780
 P 4700 4250
@@
 =1000/(2000000+2000)*650*8.2 = 2.66V differential output at 650V
 $Comp
-L R-1206 R84
+L pasv-res:R-1206 R84
 U 1 1 585AF9C1
 P 3900 3950
@@
 F 4 "CHV1206-FX-1004ELF" H 3900 3950 60  0001 C CNN "#mfg"
 F 5 "RES SMD 1k 5% [1206]" H 4650 4500 60  0001 C CNN "BOM"
+F 6 "CHV1206-FX-1004ELF" H 0   0   60  0001 C CNN "MPN"
 	1    3900 3950
 	0    1    1    0
 $EndComp
 $Comp
-L R-1206 R82
+L pasv-res:R-1206 R82
 U 1 1 585AFB0A
 P 3600 3950
@@
 F 4 "CHV1206-FX-1004ELF" H 3600 3950 60  0001 C CNN "#mfg"
 F 5 "RES SMD 1k 5% [1206]" H 4350 4500 60  0001 C CNN "BOM"
+F 6 "CHV1206-FX-1004ELF" H 0   0   60  0001 C CNN "MPN"
 	1    3600 3950
 	0    1    1    0
 $EndComp
 $Comp
-L R-0603 R85
+L pasv-res:R-0603 R85
 U 1 1 585AFCF2
 P 4400 4100
@@
 0-650V phase voltage measurement\nusing isolation amplifier
 $Comp
-L BZX84 DZ6
+L semi-diode-generic:BZX84 DZ6
 U 1 1 585B11E2
 P 4100 3600
@@
 F 3 "" H 4100 3600 60  0000 C CNN
 F 4 "BZX84-A5V1,215" H 4100 3600 60  0001 C CNN "#mfg"
+F 5 "BZX84-A5V1,215" H 0   0   60  0001 C CNN "MPN"
 	1    4100 3600
 	-1   0    0    -1
@@
 	4100 3500 4100 3450
 $Comp
-L R-0603 R83
+L pasv-res:R-0603 R83
 U 1 1 585B1392
 P 3900 3450
@@
 Connection ~ 4100 3750
 $Comp
-L C-1206 C80
+L pasv-cap:C-1206 C80
 U 1 1 585B1E88
 P 6700 3600
@@
 	6500 3750 7450 3750
 $Comp
-L C-1206 C81
+L pasv-cap:C-1206 C81
 U 1 1 585B2111
 P 7150 3600
@@
 VIN-
 $Comp
-L CONN-100MIL-F-1x1 J?
+L conn-100mil:CONN-100MIL-F-1x1 J?
 U 1 1 585BF086
 P 3200 3800
@@
 EndData
 $EndBitmap
+Wire Notes Line
+	7050 4300 7100 4300
+Wire Notes Line
+	7100 4300 7100 3900
+Wire Notes Line
+	7100 3900 7050 3900
+Text Notes 7150 4150 0    40   ~ 0
+Route very\nclose together
 $EndSCHEMATC
